Commit message: configuring transmission

File: urdf/robot.urdf.xacro (robot description, xacro)
@@ -1,5 +1,7 @@
 <?xml version="1.0"?>
 <robot xmlns:xacro="http://www.ros.org/wiki/xacro"  name="robot_arm">
+    <xacro:arg name="cmd_mode" default="position"/>
     <xacro:include filename="diff_mech.xacro"/>
     <xacro:include filename="ros2_control.xacro"/>
+    <xacro:ros2_control cmd_mode="$(arg cmd_mode)"/>
 </robot>

File: urdf/ros2_control.xacro (robot description, xacro)
@@ -1,70 +1,69 @@
 <?xml version="1.0"?>
 <robot xmlns:xacro="http://www.ros.org/wiki/xacro">
-    <xacro:arg name="cmd_mode" default="position"/>
-    <ros2_control name="StepperSystemHardware" type="system">
-        <hardware>
-            <plugin>robotic_arm/StepperSystemHardware</plugin>
-            <param name="diff_motor_L_name">diff_motor_L</param>
-            <param name="diff_motor_R_name">diff_motor_R</param>
-            <param name="device">can0</param>
-            <param name="CAN_rate">5000000</param>
-        </hardware>
-        <joint name="carrier_joint">
-            <xacro:if value="${cmd_mode == 'position'}">
-                <command_interface name="position"/>
-            </xacro:if>
-            <command_interface name="velocity"/>
-            <command_interface name="acceleration"/>
-            <state_interface name="position"/>
-            <state_interface name="velocity"/>
-        </joint>
-        <joint name="bevel_joint">
-            <xacro:if value="${cmd_mode == 'position'}">
-                <command_interface name="position"/>
-            </xacro:if>
-            <command_interface name="velocity"/>
-            <command_interface name="acceleration"/>
-            <state_interface name="position"/>
-            <state_interface name="velocity"/>
-        </joint>
-    </ros2_control>
-    <transmission name="diff_trans">
-        <type>transmission_interface/DifferentialTransmission</type>
-        <actuator name="diff_motor_L">
-            <xacro:if value="${cmd_mode == 'position'}">
-                <hardwareInterface>hardware_interface/PositionJointInterface</hardwareInterface>
-            </xacro:if>
-            <xacro:if value="${cmd_mode == 'speed'}">
-                <hardwareInterface>hardware_interface/VelocityJointInterface</hardwareInterface>
-            </xacro:if>
-            <mechanicalReduction>1</mechanicalReduction>
-        </actuator>
-        <actuator name="diff_motor_R">
-            <xacro:if value="${cmd_mode == 'position'}">
-                <hardwareInterface>hardware_interface/PositionJointInterface</hardwareInterface>
-            </xacro:if>
-            <xacro:if value="${cmd_mode == 'speed'}">
-                <hardwareInterface>hardware_interface/VelocityJointInterface</hardwareInterface>
-            </xacro:if>
-            <mechanicalReduction>1</mechanicalReduction>
-        </actuator>
-        <joint name="carrier_joint">
-            <xacro:if value="${cmd_mode == 'position'}">
-                <hardwareInterface>hardware_interface/PositionJointInterface</hardwareInterface>
-            </xacro:if>
-            <xacro:if value="${cmd_mode == 'speed'}">
-                <hardwareInterface>hardware_interface/VelocityJointInterface</hardwareInterface>
-            </xacro:if>
-            <role>sum</role>
-        </joint>
-        <joint name="bevel_joint">
-            <xacro:if value="${cmd_mode == 'position'}">
-                <hardwareInterface>hardware_interface/PositionJointInterface</hardwareInterface>
-            </xacro:if>
-            <xacro:if value="${cmd_mode == 'speed'}">
-                <hardwareInterface>hardware_interface/VelocityJointInterface</hardwareInterface>
-            </xacro:if>
-            <role>diff</role>
-        </joint>
-    </transmission>
+    <xacro:macro name="ros2_control" params="cmd_mode">
+        <ros2_control name="StepperSystemHardware" type="system">
+            <hardware>
+                <plugin>robotic_arm/StepperSystemHardware</plugin>
+                <param name="diff_motor_L_name">diff_motor_L</param>
+                <param name="diff_motor_R_name">diff_motor_R</param>
+                <param name="device">can0</param>
+                <param name="CAN_rate">5000000</param>
+            </hardware>
+            <joint name="carrier_joint">
+                <xacro:if value="${cmd_mode == 'position'}">
+                    <command_interface name="position"/>
+                </xacro:if>
+                <command_interface name="velocity"/>
+                <command_interface name="acceleration"/>
+                <state_interface name="position"/>
+                <state_interface name="velocity"/>
+            </joint>
+            <joint name="bevel_joint">
+                <xacro:if value="${cmd_mode == 'position'}">
+                    <command_interface name="position"/>
+                </xacro:if>
+                <command_interface name="velocity"/>
+                <command_interface name="acceleration"/>
+                <state_interface name="position"/>
+                <state_interface name="velocity"/>
+            </joint>
+            <transmission name="diff_trans">
+                <plugin>transmission_interface/DifferentialTransmission</plugin>
+                <actuator name="diff_motor_L" role="actuator1">
+                    <xacro:if value="${cmd_mode == 'position'}">
+                        <hardwareInterface>hardware_interface/PositionJointInterface</hardwareInterface>
+                    </xacro:if>
+                    <xacro:if value="${cmd_mode == 'speed'}">
+                        <hardwareInterface>hardware_interface/VelocityJointInterface</hardwareInterface>
+                    </xacro:if>
+                    <mechanicalReduction>1</mechanicalReduction>
+                </actuator>
+                <actuator name="diff_motor_R" role="actuator2">
+                    <xacro:if value="${cmd_mode == 'position'}">
+                        <hardwareInterface>hardware_interface/PositionJointInterface</hardwareInterface>
+                    </xacro:if>
+                    <xacro:if value="${cmd_mode == 'speed'}">
+                        <hardwareInterface>hardware_interface/VelocityJointInterface</hardwareInterface>
+                    </xacro:if>
+                    <mechanicalReduction>1</mechanicalReduction>
+                </actuator>
+                <joint name="carrier_joint" role="joint1">
+                    <xacro:if value="${cmd_mode == 'position'}">
+                        <hardwareInterface>hardware_interface/PositionJointInterface</hardwareInterface>
+                    </xacro:if>
+                    <xacro:if value="${cmd_mode == 'speed'}">
+                        <hardwareInterface>hardware_interface/VelocityJointInterface</hardwareInterface>
+                    </xacro:if>
+                </joint>
+                <joint name="bevel_joint" role="joint2">
+                    <xacro:if value="${cmd_mode == 'position'}">
+                        <hardwareInterface>hardware_interface/PositionJointInterface</hardwareInterface>
+                    </xacro:if>
+                    <xacro:if value="${cmd_mode == 'speed'}">
+                        <hardwareInterface>hardware_interface/VelocityJointInterface</hardwareInterface>
+                    </xacro:if>
+                </joint>
+            </transmission>
+        </ros2_control>
+    </xacro:macro>
 </robot>

Commit message: configuring trajectory controllers

File: urdf/robot.urdf.xacro (robot description, xacro)
@@ -10,4 +10,5 @@
     <xacro:unless value="$(arg real_time)">
         <xacro:include filename="sim_control.xacro"/>
+        <xacro:ros2_control_mock_hardware cmd_mode="$(arg cmd_mode)"/>
     </xacro:unless>
 </robot>

File: urdf/ros2_control.xacro (robot description, xacro)
@@ -8,5 +8,5 @@
                 <param name="central_bevel_name">bevel_joint</param>
                 <param name="device">can0</param>
-                <param name="CAN_rate">5000000</param>
+                <param name="CAN_rate">500000</param>
                 <param name="timeout_ms">5000</param>
             </hardware>

File: urdf/sim_control.xacro (robot description, xacro)
@@ -1,4 +1,5 @@
 <?xml version="1.0"?>
 <robot xmlns:xacro="http://www.ros.org/wiki/xacro">
+  <xacro:macro name="ros2_control_mock_hardware" params="cmd_mode">
     <ros2_control name="sim_control" type="system">
       <hardware>
@@ -6,5 +7,7 @@
       </hardware>
       <joint name="carrier_joint">
-        <command_interface name="position"/>
+        <xacro:if value="${cmd_mode == 'position'}">
+          <command_interface name="position"/>
+        </xacro:if>
         <command_interface name="velocity"/>
         <command_interface name="acceleration"/>
@@ -15,5 +18,7 @@
       </joint>
       <joint name="bevel_joint">
-        <command_interface name="position"/>
+        <xacro:if value="${cmd_mode == 'position'}">
+          <command_interface name="position"/>
+        </xacro:if>
         <command_interface name="velocity"/>
         <command_interface name="acceleration"/>
@@ -24,3 +29,4 @@
       </joint>
     </ros2_control>
+  </xacro:macro>
 </robot>
