Commit message: merged new changes from improved hardware_interface

File: urdf/robot.urdf.xacro (robot description, xacro)
@@ -1,14 +1,10 @@
 <?xml version="1.0"?>
-<robot xmlns:xacro="http://www.ros.org/wiki/xacro"  name="robot_arm">
+<robot xmlns:xacro="http://www.ros.org/wiki/xacro"  name="robotic_arm">
     <xacro:arg name="cmd_mode" default="position"/>
-    <xacro:arg name="real_time" default="true"/>
+    <xacro:arg name="HW_mode" default="mock"/>
     <xacro:include filename="robot_core.xacro"/>
-    <xacro:if value="$(arg real_time)">
-        <xacro:include filename="ros2_control.xacro"/>
-        <xacro:ros2_control cmd_mode="$(arg cmd_mode)"/>
-    </xacro:if>
-    <xacro:unless value="$(arg real_time)">
-        <xacro:include filename="sim_control.xacro"/>
-        <xacro:ros2_control_mock_hardware cmd_mode="$(arg cmd_mode)"/>
-    </xacro:unless>
+    <xacro:include filename="gazebo.xacro"/>
+    <xacro:include filename="ros2_control.xacro"/>
+    <!-- XACRO to handle multiple ros2_control hardware_interface plugins -->
+    <xacro:ros2_control HW_mode="$(arg HW_mode)" cmd_mode="$(arg cmd_mode)"/>
 </robot>

File: urdf/robot_core.xacro (robot description, xacro)
@@ -30,4 +30,9 @@
             </geometry>
         </collision>
+        <inertial>
+            <origin xyz="0 0 0.0225" rpy="0 0 0"/>
+            <mass value="0.5"/>
+            <inertia ixx="0.001" ixy="0.0" ixz="0.0" iyy="0.001" iyz="0.0" izz="0.001"/>
+        </inertial>
     </link>
     <link name="top_base">
@@ -45,4 +50,9 @@
             </geometry>
         </collision>
+        <inertial>
+            <origin xyz="0 0 0.1" rpy="0 0 0"/>
+            <mass value="0.8"/>
+            <inertia ixx="0.002" ixy="0.0" ixz="0.0" iyy="0.002" iyz="0.0" izz="0.001"/>
+        </inertial>
     </link>
     <joint name="bottom_base_joint" type="fixed">
@@ -75,4 +85,9 @@
             </geometry>
         </collision>
+        <inertial>
+            <origin xyz="0.03615 0 0.20655" rpy="0 0 0"/>
+            <mass value="0.6"/>
+            <inertia ixx="0.003" ixy="0.0" ixz="0.0" iyy="0.003" iyz="0.0" izz="0.0005"/>
+        </inertial>
     </link>
     <joint name="shoulder_joint" type="revolute">
@@ -100,4 +115,9 @@
             </geometry>
         </collision>
+        <inertial>
+            <origin xyz="-0.00475 0.055 0.0556" rpy="0 0 0"/>
+            <mass value="0.5"/>
+            <inertia ixx="0.001" ixy="0.0" ixz="0.0" iyy="0.001" iyz="0.0" izz="0.0005"/>
+        </inertial>
     </link>
     <joint name="elbow_joint" type="revolute">
@@ -125,4 +145,9 @@
             </geometry>
         </collision>
+        <inertial>
+            <origin xyz="0 0.128 0" rpy="-${pi/2} 0 0"/>
+            <mass value="0.4"/>
+            <inertia ixx="0.001" ixy="0.0" ixz="0.0" iyy="0.0005" iyz="0.0" izz="0.001"/>
+        </inertial>
     </link>
     <joint name="forearm_joint" type="revolute">
@@ -147,4 +172,9 @@
             </geometry>
         </collision>
+        <inertial>
+            <origin xyz="0 0 0.01995" rpy="0 0 0"/>
+            <mass value="0.2"/>
+            <inertia ixx="0.0001" ixy="0.0" ixz="0.0" iyy="0.0001" iyz="0.0" izz="0.0001"/>
+        </inertial>
     </link>
     <joint name="wrist_carrier_joint" type="revolute">
@@ -169,4 +199,9 @@
             </geometry>
         </collision>
+        <inertial>
+            <origin xyz="0 0 0" rpy="0 0 0"/>
+            <mass value="0.1"/>
+            <inertia ixx="0.0001" ixy="0.0" ixz="0.0" iyy="0.0001" iyz="0.0" izz="0.0001"/>
+        </inertial>
     </link>
     <joint name="wrist_bevel_joint" type="revolute">
@@ -177,3 +212,6 @@
         <limit lower="-${pi}" upper="${pi}" effort="100" velocity="1"/>
     </joint>
+    <!-- ****************************************************************************************** -->
+    <!-- **************************************** Claw ******************************************** -->
+    <!-- ****************************************************************************************** -->
 </robot>

File: urdf/ros2_control.xacro (robot description, xacro)
@@ -1,88 +1,212 @@
 <?xml version="1.0"?>
 <robot xmlns:xacro="http://www.ros.org/wiki/xacro">
-    <xacro:macro name="ros2_control" params="cmd_mode">
-        <ros2_control name="StepperSystemHardware" type="system">
-            <hardware>
-                <plugin>robotic_arm/StepperSystemHardware</plugin>
-                <param name="base_name">base_joint</param>
-                <param name="base_joint_reduction">16</param>
-                <param name="shoulder_name">shoulder_joint</param>
-                <param name="shoulder_joint_reduction">16</param>
-                <param name="elbow_name">elbow_joint</param>
-                <param name="elbow_joint_reduction">16</param>
-                <param name="forearm_name">forearm_joint</param>
-                <param name="forearm_joint_reduction">16</param>
-                <param name="wrist_carrier_name">wrist_carrier_joint</param>
-                <param name="wrist_bevel_name">wrist_bevel_joint</param>
-                <param name="wrsit_carrier_joint_reduction">16</param>
-                <param name="wrist_bevel_joint_reduction">16</param>
-                <param name="device">can0</param>
-                <param name="CAN_rate">500000</param>
-            </hardware>
-            <joint name="base_joint">
-                <xacro:if value="${cmd_mode == 'position'}">
-                    <command_interface name="position"/>
-                </xacro:if>
-                <command_interface name="velocity"/>
-                <command_interface name="acceleration"/>
-                <state_interface name="position"/>
-                <state_interface name="velocity"/>
-            </joint>
-            <joint name="shoulder_joint">
-                <xacro:if value="${cmd_mode == 'position'}">
-                    <command_interface name="position"/>
-                </xacro:if>
-                <command_interface name="velocity"/>
-                <command_interface name="acceleration"/>
-                <state_interface name="position"/>
-                <state_interface name="velocity"/>
-            </joint>
-            <joint name="elbow_joint">
-                <xacro:if value="${cmd_mode == 'position'}">
-                    <command_interface name="position"/>
-                </xacro:if>
-                <command_interface name="velocity"/>
-                <command_interface name="acceleration"/>
-                <state_interface name="position"/>
-                <state_interface name="velocity"/>
-            </joint>
-            <joint name="forearm_joint">
-                <xacro:if value="${cmd_mode == 'position'}">
-                    <command_interface name="position"/>
-                </xacro:if>
-                <command_interface name="velocity"/>
-                <command_interface name="acceleration"/>
-                <state_interface name="position"/>
-                <state_interface name="velocity"/>
-            </joint>
-            <joint name="bevel_joint">
-                <xacro:if value="${cmd_mode == 'position'}">
-                    <command_interface name="position"/>
-                </xacro:if>
-                <command_interface name="velocity"/>
-                <command_interface name="acceleration"/>
-                <state_interface name="position"/>
-                <state_interface name="velocity"/>
-            </joint>
-        </ros2_control>
-            <joint name="wrist_carrier_joint">
-                <xacro:if value="${cmd_mode == 'position'}">
-                    <command_interface name="position"/>
-                </xacro:if>
-                <command_interface name="velocity"/>
-                <command_interface name="acceleration"/>
-                <state_interface name="position"/>
-                <state_interface name="velocity"/>
-            </joint>
-            <joint name="wrist_bevel_joint">
-                <xacro:if value="${cmd_mode == 'position'}">
-                    <command_interface name="position"/>
-                </xacro:if>
-                <command_interface name="velocity"/>
-                <command_interface name="acceleration"/>
-                <state_interface name="position"/>
-                <state_interface name="velocity"/>
-            </joint>
-        </ros2_control>
+    <xacro:macro name="ros2_control" params="HW_mode cmd_mode">
+        <xacro:if value="${HW_mode == 'real'}">
+            <ros2_control name="StepperSystemHardware" type="system">
+                <hardware>
+                    <plugin>robotic_arm/StepperSystemHardware</plugin>
+                    <param name="device">can0</param>
+                    <param name="CAN_rate">500000</param>
+                    <param name="timeout">5</param>
+                    <param name="loop_rate">1000</param>
+                </hardware>
+                <joint name="base_joint">
+                    <xacro:if value="${cmd_mode == 'position'}">
+                        <command_interface name="position"/>
+                    </xacro:if>
+                    <command_interface name="velocity"/>
+                    <command_interface name="acceleration"/>
+                    <state_interface name="position"/>
+                    <state_interface name="velocity"/>
+                    <param name="reduction">1.0</param>
+                    <param name="CAN_id">0x01</param>
+                </joint>
+                <joint name="shoulder_joint">
+                    <xacro:if value="${cmd_mode == 'position'}">
+                        <command_interface name="position"/>
+                    </xacro:if>
+                    <command_interface name="velocity"/>
+                    <command_interface name="acceleration"/>
+                    <state_interface name="position"/>
+                    <state_interface name="velocity"/>
+                    <param name="reduction">16.0</param>
+                    <param name="CAN_id">0x02</param>
+                </joint>
+                <joint name="elbow_joint">
+                    <xacro:if value="${cmd_mode == 'position'}">
+                        <command_interface name="position"/>
+                    </xacro:if>
+                    <command_interface name="velocity"/>
+                    <command_interface name="acceleration"/>
+                    <state_interface name="position"/>
+                    <state_interface name="velocity"/>
+                    <param name="reduction">16.0</param>
+                    <param name="CAN_id">0x03</param>
+                </joint>
+                <joint name="forearm_joint">
+                    <xacro:if value="${cmd_mode == 'position'}">
+                        <command_interface name="position"/>
+                    </xacro:if>
+                    <command_interface name="velocity"/>
+                    <command_interface name="acceleration"/>
+                    <state_interface name="position"/>
+                    <state_interface name="velocity"/>
+                    <param name="reduction">16.0</param>
+                    <param name="CAN_id">0x04</param>
+                </joint>
+                <joint name="wrist_carrier_joint">
+                    <xacro:if value="${cmd_mode == 'position'}">
+                        <command_interface name="position"/>
+                    </xacro:if>
+                    <command_interface name="velocity"/>
+                    <command_interface name="acceleration"/>
+                    <state_interface name="position"/>
+                    <state_interface name="velocity"/>
+                    <param name="reduction">2.0</param>
+                    <param name="CAN_id">0x05</param>
+                </joint>
+                <joint name="wrist_bevel_joint">
+                    <xacro:if value="${cmd_mode == 'position'}">
+                        <command_interface name="position"/>
+                    </xacro:if>
+                    <command_interface name="velocity"/>
+                    <command_interface name="acceleration"/>
+                    <state_interface name="position"/>
+                    <state_interface name="velocity"/>
+                    <param name="reduction">2.0</param>
+                    <param name="CAN_id">0x06</param>
+                </joint>
+            </ros2_control>
+        </xacro:if>
+        <xacro:if value="${HW_mode == 'gazebo'}">
+            <ros2_control name="GazeboSimSystem" type="system">
+                <hardware>
+                    <plugin>gazebo_ros2_control/GazeboSystem</plugin>
+                </hardware>
+                <joint name="base_joint">
+                    <xacro:if value="${cmd_mode == 'position'}">
+                        <command_interface name="position"/>
+                    </xacro:if>
+                    <command_interface name="velocity"/>
+                    <command_interface name="acceleration"/>
+                    <state_interface name="position"/>
+                    <state_interface name="velocity"/>
+                </joint>
+                <joint name="shoulder_joint">
+                    <xacro:if value="${cmd_mode == 'position'}">
+                        <command_interface name="position"/>
+                    </xacro:if>
+                    <command_interface name="velocity"/>
+                    <command_interface name="acceleration"/>
+                    <state_interface name="position"/>
+                    <state_interface name="velocity"/>
+                </joint>
+                <joint name="elbow_joint">
+                    <xacro:if value="${cmd_mode == 'position'}">
+                        <command_interface name="position"/>
+                    </xacro:if>
+                    <command_interface name="velocity"/>
+                    <command_interface name="acceleration"/>
+                    <state_interface name="position"/>
+                    <state_interface name="velocity"/>
+                </joint>
+                <joint name="forearm_joint">
+                    <xacro:if value="${cmd_mode == 'position'}">
+                        <command_interface name="position"/>
+                    </xacro:if>
+                    <command_interface name="velocity"/>
+                    <command_interface name="acceleration"/>
+                    <state_interface name="position"/>
+                    <state_interface name="velocity"/>
+                </joint>
+                <joint name="wrist_carrier_joint">
+                    <xacro:if value="${cmd_mode == 'position'}">
+                        <command_interface name="position"/>
+                    </xacro:if>
+                    <command_interface name="velocity"/>
+                    <command_interface name="acceleration"/>
+                    <state_interface name="position">
+                        <param name="initial_value">0.0</param>
+                    </state_interface>
+                    <state_interface name="velocity"/>
+                </joint>
+                <joint name="wrist_bevel_joint">
+                    <xacro:if value="${cmd_mode == 'position'}">
+                        <command_interface name="position"/>
+                    </xacro:if>
+                    <command_interface name="velocity"/>
+                    <command_interface name="acceleration"/>
+                    <state_interface name="position">
+                        <param name="initial_value">0.0</param>
+                    </state_interface>
+                    <state_interface name="velocity"/>
+                </joint>
+            </ros2_control>
+        </xacro:if>
+        <xacro:if value="${HW_mode == 'mock'}">
+            <ros2_control name="sim_control" type="system">
+                <hardware>
+                    <plugin>mock_components/GenericSystem</plugin>
+                </hardware>
+                <joint name="base_joint">
+                    <xacro:if value="${cmd_mode == 'position'}">
+                        <command_interface name="position"/>
+                    </xacro:if>
+                    <command_interface name="velocity"/>
+                    <command_interface name="acceleration"/>
+                    <state_interface name="position"/>
+                    <state_interface name="velocity"/>
+                </joint>
+                <joint name="shoulder_joint">
+                    <xacro:if value="${cmd_mode == 'position'}">
+                        <command_interface name="position"/>
+                    </xacro:if>
+                    <command_interface name="velocity"/>
+                    <command_interface name="acceleration"/>
+                    <state_interface name="position"/>
+                    <state_interface name="velocity"/>
+                </joint>
+                <joint name="elbow_joint">
+                    <xacro:if value="${cmd_mode == 'position'}">
+                        <command_interface name="position"/>
+                    </xacro:if>
+                    <command_interface name="velocity"/>
+                    <command_interface name="acceleration"/>
+                    <state_interface name="position"/>
+                    <state_interface name="velocity"/>
+                </joint>
+                <joint name="forearm_joint">
+                    <xacro:if value="${cmd_mode == 'position'}">
+                        <command_interface name="position"/>
+                    </xacro:if>
+                    <command_interface name="velocity"/>
+                    <command_interface name="acceleration"/>
+                    <state_interface name="position"/>
+                    <state_interface name="velocity"/>
+                </joint>
+                <joint name="wrist_carrier_joint">
+                    <xacro:if value="${cmd_mode == 'position'}">
+                        <command_interface name="position"/>
+                    </xacro:if>
+                    <command_interface name="velocity"/>
+                    <command_interface name="acceleration"/>
+                    <state_interface name="position">
+                    <param name="initial_value">0.0</param>
+                    </state_interface>
+                    <state_interface name="velocity"/>
+                </joint>
+                <joint name="wrist_bevel_joint">
+                    <xacro:if value="${cmd_mode == 'position'}">
+                        <command_interface name="position"/>
+                    </xacro:if>
+                    <command_interface name="velocity"/>
+                    <command_interface name="acceleration"/>
+                    <state_interface name="position">
+                    <param name="initial_value">0.0</param>
+                    </state_interface>
+                    <state_interface name="velocity"/>
+                </joint>
+            </ros2_control>
+        </xacro:if>
     </xacro:macro>
 </robot>
