Commit message: 6-DOF added to urdf

File: urdf/robot_core.xacro (robot description, xacro)
@@ -79,6 +79,6 @@
         <parent link="top_base"/>
         <child link="shoulder"/>
-        <origin xyz="-0.0655 0.13558 0.1998" rpy="${pi/2} 0 -${pi/2}"/>
-        <axis xyz="0 0 1"/>
+        <origin xyz="-0.0655 0.13558 0.1998" rpy="0 0 0"/>
+        <axis xyz="-1 0 0"/>
         <limit lower="-${3*pi/4}" upper="${3*pi/4}" effort="100" velocity="1"/>
     </joint>
@@ -104,5 +104,74 @@
         <parent link="shoulder"/>
         <child link="elbow"/>
-        <origin xyz="0.0068 0.13552 0.61294" rpy="0 0 0"/>
+        <origin xyz="0.0723 0 0.4131" rpy="0 0 0"/>
+        <axis xyz="-1 0 0"/>
+        <limit lower="-${pi}" upper="${pi}" effort="100" velocity="1"/>
+    </joint>
+    <!-- ****************************************************************************************** -->
+    <!-- *************************************** Wrist ******************************************** -->
+    <!-- ****************************************************************************************** -->
+    <link name="forearm">
+        <visual>
+            <origin xyz="0 0 0" rpy="-${pi/2} 0 0"/>
+            <geometry>
+                <mesh filename="package://robotic_arm/meshes/forearm.stl" scale="${scale_factor}"/>
+            </geometry>
+            <material name="grey"/>
+        </visual>
+        <collision>
+            <origin xyz="0 0 0"/>
+            <geometry>
+                <mesh filename="package://robotic_arm/meshes/forearm.stl" scale="${scale_factor}"/>
+            </geometry>
+        </collision>
+    </link>
+    <joint name="forearm_joint" type="revolute">
+        <parent link="elbow"/>
+        <child link="forearm"/>
+        <origin xyz="-0.0095 0.110 0.1112" rpy="0 0 0"/>
+        <axis xyz="0 1 0"/>
+        <limit lower="-${pi}" upper="${pi}" effort="100" velocity="1"/>
+    </joint>
+    <link name="wrist_carrier">
+        <visual>
+            <origin xyz="0 0 0"/>
+            <geometry>
+                <mesh filename="package://robotic_arm/meshes/wrist_carrier.stl" scale="${scale_factor}"/>
+            </geometry>
+            <material name="blue"/>
+        </visual>
+        <collision>
+            <origin xyz="0 0 0"/>
+            <geometry>
+                <mesh filename="package://robotic_arm/meshes/wrist_carrier.stl" scale="${scale_factor}"/>
+            </geometry>
+        </collision>
+    </link>
+    <joint name="wrist_carrier_joint" type="revolute">
+        <parent link="forearm"/>
+        <child link="wrist_carrier"/>
+        <origin xyz="0 0.256 0" rpy="-${pi/2} 0 0"/>
+        <axis xyz="1 0 0"/>
+        <limit lower="-${3*pi/4}" upper="${3*pi/4}" effort="100" velocity="1"/>
+    </joint>
+    <link name="wrist_bevel">
+        <visual>
+            <origin xyz="0 0 0" />
+            <geometry>
+                <mesh filename="package://robotic_arm/meshes/wrist_bevel.stl" scale="${scale_factor}"/>
+            </geometry>
+            <material name="grey"/>
+        </visual>
+        <collision>
+            <origin xyz="0 0 0"/>
+            <geometry>
+                <mesh filename="package://robotic_arm/meshes/wrist_bevel.stl" scale="${scale_factor}"/>
+            </geometry>
+        </collision>
+    </link>
+    <joint name="wrist_bevel_joint" type="revolute">
+        <parent link="wrist_carrier"/>
+        <child link="wrist_bevel"/>
+        <origin xyz="0 0 0.0399" rpy="0 0 0"/>
         <axis xyz="0 0 1"/>
         <limit lower="-${pi}" upper="${pi}" effort="100" velocity="1"/>

Commit message: joint to motor mappings added

File: urdf/robot_core.xacro (robot description, xacro)
@@ -46,10 +46,10 @@
         </collision>
     </link>
-    <joint name="base_joint" type="fixed">
+    <joint name="bottom_base_joint" type="fixed">
         <parent link="world"/>
         <child link="bottom_base"/>
         <origin xyz="0 0 0" rpy="0 0 0"/>
     </joint>
-    <joint name="top_base_joint" type="revolute">
+    <joint name="base_joint" type="revolute">
         <parent link="bottom_base"/>
         <child link="top_base"/>

File: urdf/ros2_control.xacro (robot description, xacro)
@@ -5,11 +5,47 @@
             <hardware>
                 <plugin>robotic_arm/StepperSystemHardware</plugin>
-                <param name="carrier_name">carrier_joint</param>
-                <param name="central_bevel_name">bevel_joint</param>
+                <param name="base_name">base_joint</param>
+                <param name="base_joint_reduction">16</param>
+                <param name="shoulder_name">shoulder_joint</param>
+                <param name="shoulder_joint_reduction">16</param>
+                <param name="elbow_name">elbow_joint</param>
+                <param name="elbow_joint_reduction">16</param>
+                <param name="forearm_name">forearm_joint</param>
+                <param name="forearm_joint_reduction">16</param>
+                <param name="wrist_carrier_name">wrist_carrier_joint</param>
+                <param name="wrist_bevel_name">wrist_bevel_joint</param>
+                <param name="wrsit_carrier_joint_reduction">16</param>
+                <param name="wrist_bevel_joint_reduction">16</param>
                 <param name="device">can0</param>
                 <param name="CAN_rate">500000</param>
-                <param name="timeout_ms">5000</param>
             </hardware>
-            <joint name="carrier_joint">
+            <joint name="base_joint">
+                <xacro:if value="${cmd_mode == 'position'}">
+                    <command_interface name="position"/>
+                </xacro:if>
+                <command_interface name="velocity"/>
+                <command_interface name="acceleration"/>
+                <state_interface name="position"/>
+                <state_interface name="velocity"/>
+            </joint>
+            <joint name="shoulder_joint">
+                <xacro:if value="${cmd_mode == 'position'}">
+                    <command_interface name="position"/>
+                </xacro:if>
+                <command_interface name="velocity"/>
+                <command_interface name="acceleration"/>
+                <state_interface name="position"/>
+                <state_interface name="velocity"/>
+            </joint>
+            <joint name="elbow_joint">
+                <xacro:if value="${cmd_mode == 'position'}">
+                    <command_interface name="position"/>
+                </xacro:if>
+                <command_interface name="velocity"/>
+                <command_interface name="acceleration"/>
+                <state_interface name="position"/>
+                <state_interface name="velocity"/>
+            </joint>
+            <joint name="forearm_joint">
                 <xacro:if value="${cmd_mode == 'position'}">
                     <command_interface name="position"/>
@@ -30,4 +66,23 @@
             </joint>
         </ros2_control>
+            <joint name="wrist_carrier_joint">
+                <xacro:if value="${cmd_mode == 'position'}">
+                    <command_interface name="position"/>
+                </xacro:if>
+                <command_interface name="velocity"/>
+                <command_interface name="acceleration"/>
+                <state_interface name="position"/>
+                <state_interface name="velocity"/>
+            </joint>
+            <joint name="wrist_bevel_joint">
+                <xacro:if value="${cmd_mode == 'position'}">
+                    <command_interface name="position"/>
+                </xacro:if>
+                <command_interface name="velocity"/>
+                <command_interface name="acceleration"/>
+                <state_interface name="position"/>
+                <state_interface name="velocity"/>
+            </joint>
+        </ros2_control>
     </xacro:macro>
 </robot>

Commit message: improving joint self collisions

File: urdf/robot_core.xacro (robot description, xacro)
@@ -215,3 +215,83 @@
     <!-- **************************************** Claw ******************************************** -->
     <!-- ****************************************************************************************** -->
+    <link name="claw_base">
+        <visual>
+            <origin xyz="-0.04 -0.025 0" />
+            <geometry>
+                <mesh filename="package://robotic_arm/meshes/claw_base.stl" scale="${scale_factor}"/>
+            </geometry>
+            <material name="grey"/>
+        </visual>
+        <collision>
+            <origin xyz="0 0 0"/>
+            <geometry>
+                <mesh filename="package://robotic_arm/meshes/claw_base.stl" scale="${scale_factor}"/>
+            </geometry>
+        </collision>
+        <inertial>
+            <origin xyz="0 0 0.02" rpy="0 0 0"/>
+            <mass value="0.1"/>
+            <inertia ixx="0.0001" ixy="0.0" ixz="0.0" iyy="0.0001" iyz="0.0" izz="0.0001"/>
+        </inertial>
+    </link>
+    <joint name="claw_base_joint" type="fixed">
+        <parent link="wrist_bevel"/>
+        <child link="claw_base"/>
+        <origin xyz="0 0 0" rpy="0 0 0"/>
+    </joint>
+        <link name="right_claw">
+        <visual>
+            <origin xyz="0 0 -0.015" />
+            <geometry>
+                <mesh filename="package://robotic_arm/meshes/claw_right.stl" scale="${scale_factor}"/>
+            </geometry>
+            <material name="grey"/>
+        </visual>
+        <collision>
+            <origin xyz="0 0 0"/>
+            <geometry>
+                <mesh filename="package://robotic_arm/meshes/claw_right.stl" scale="${scale_factor}"/>
+            </geometry>
+        </collision>
+        <inertial>
+            <origin xyz="0 -0.02 0" rpy="0 0 0"/>
+            <mass value="0.05"/>
+            <inertia ixx="0.00005" ixy="0.0" ixz="0.0" iyy="0.00005" iyz="0.0" izz="0.00005"/>
+        </inertial>
+    </link>
+    <joint name="right_claw_joint" type="prismatic">
+        <parent link="claw_base"/>
+        <child link="right_claw"/>
+        <origin xyz="0 0 0.03" rpy="${pi/2} 0 0"/>
+        <axis xyz="1 0 0"/>
+        <limit lower="0" upper="0.03" effort="100" velocity="1"/>
+    </joint>
+    <link name="left_claw">
+        <visual>
+            <origin xyz="0 0 -0.015" />
+            <geometry>
+                <mesh filename="package://robotic_arm/meshes/claw_left.stl" scale="${scale_factor}"/>
+            </geometry>
+            <material name="grey"/>
+        </visual>
+        <collision>
+            <origin xyz="0 0 0"/>
+            <geometry>
+                <mesh filename="package://robotic_arm/meshes/claw_left.stl" scale="${scale_factor}"/>
+            </geometry>
+        </collision>
+        <inertial>
+            <origin xyz="0 0.02 0" rpy="0 0 0"/>
+            <mass value="0.05"/>
+            <inertia ixx="0.00005" ixy="0.0" ixz="0.0" iyy="0.00005" iyz="0.0" izz="0.00005"/>
+        </inertial>
+    </link>
+    <joint name="left_claw_joint" type="prismatic">
+        <parent link="claw_base"/>
+        <child link="left_claw"/>
+        <origin xyz="0 0 0.03" rpy="${pi/2} 0 0"/>
+        <axis xyz="1 0 0"/>
+        <limit lower="-0.03" upper="0" effort="100" velocity="1"/>
+        <mimic joint="right_claw_joint" multiplier="-1"/>
+    </joint>
 </robot>
